File: turbidity/basic-handheld-turbidimeter/hardware/basic-handheld-turbidimeter.sch (EAGLE design)
At the start: 33 parts, among them Q1 16.000, U1 ATMEGA328P-PU

Commit message: added OSHW logo to main board, added seven segment helper board
Parts:
- 2.4V_ZENER: value DIODE-ZENERPTH -> DNP
Changed lines of the file:
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@@
 <?xml version="1.0" encoding="utf-8"?>
 <!DOCTYPE eagle SYSTEM "eagle.dtd">
-<eagle version="7.1.0">
+<eagle version="7.3.0">
 <drawing>
 <settings>
@@
 <part name="SUPPLY5" library="supply2" deviceset="GND" device=""/>
 <part name="SUPPLY15" library="supply2" deviceset="GND" device=""/>
-<part name="2.4V_ZENER" library="SparkFun-DiscreteSemi" deviceset="DIODE-ZENER" device="PTH"/>
+<part name="2.4V_ZENER" library="SparkFun-DiscreteSemi" deviceset="DIODE-ZENER" device="PTH" value="DNP"/>
 <part name="R10" library="rcl" deviceset="R-US_" device="0207/12" value="220"/>
 <part name="LIPO" library="pinhead" deviceset="PINHD-1X2" device=""/>

Commit message: added current regulator for IR LED
Parts:
- removed 2.4V_ZENER: DNP, SparkFun-DiscreteSemi:DIODE-ZENERPTH
- added U$6: AL5809, awqua_eagle_library:AL5809
Connections:
- new net N$2: R10.2, U$6.OUT
- net GND: no longer 2.4V_ZENER.A
- net LED: no longer 2.4V_ZENER.C
- net PD4: now also U$6.IN; no longer R10.2
Other:
- moved on the sheet: LED, R10
