File: temperature/basic-thermometer/hardware/basic-thermometer-SD.brd (EAGLE design)
At the start: 22.9 x 30.5 mm, 20 parts, among them IC1 MEGA8-AI

Commit message: update to basic-thermometer-SD
Parts:
- added C4: 100n, SparkFun:0603-CAP
- moved C5 7.13 mm to (7.62, 9.84), turned to 180 degrees
- moved C8 6.84 mm to (14.6, 9.84), turned to 0 degrees
- moved C3 1.27 mm to (17.5, 27.0), turned to 270 degrees
- flipped JP3 to the top
Connections:
- removed net AVCC: IC1.18
- net GND: now also C4.1
- net PD2: now also JP5.1
- net PD5: now also C3.2, JP6.3
- net VCC: now also C4.2, IC1.18; no longer C3.2, JP6.3
Routing:
- net VCC: track 117.5 -> 80.8 mm
- net GND: track 142.9 -> 107.4 mm, vias 1 -> 2
- net PD5: track 0.00 -> 21.2 mm, vias 0 -> 2
- net PD2: track 0.00 -> 12.2 mm
- net RST: track 30.7 -> 21.9 mm
- net AREF: track 14.4 -> 23.0 mm
- net SCL: track 34.1 -> 39.5 mm
- net SDA: track 48.0 -> 43.2 mm
- net TX: track 21.9 -> 17.3 mm
- net PD6: track 11.6 -> 15.5 mm, vias 0 -> 2
- net SCK: track 27.4 -> 23.7 mm
- net MISO: track 23.2 -> 20.3 mm, vias 0 -> 1
- net RX: track 19.0 -> 18.6 mm, vias 2 -> 1
- net MOSI: vias 0 -> 1
- added copper zone on layer 1, net GND
