File: turbidity/devices/basic-handheld-turbidimeter/hardware/basic-handheld-turbidimeter.brd (EAGLE design)
At the start: 45.1 x 63.5 mm, 38 parts, among them Q1 16.000, U1 ATMEGA328P-PU

Commit message: updating pdfs of board and schematic
Other:
- board text added: "Released under Creative Commons license BY-SA 4.0 https://creativecommons.org/licenses/by-sa/4.0"
Changed lines of the file:
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@@
 <?xml version="1.0" encoding="utf-8"?>
 <!DOCTYPE eagle SYSTEM "eagle.dtd">
-<eagle version="6.5.0">
+<eagle version="7.3.0">
 <drawing>
 <settings>
@@
 <layer number="46" name="Milling" color="3" fill="1" visible="no" active="yes"/>
 <layer number="47" name="Measures" color="7" fill="1" visible="no" active="yes"/>
-<layer number="48" name="Document" color="7" fill="1" visible="no" active="yes"/>
+<layer number="48" name="Document" color="7" fill="1" visible="yes" active="yes"/>
 <layer number="49" name="Reference" color="7" fill="1" visible="no" active="yes"/>
 <layer number="50" name="dxf" color="7" fill="1" visible="no" active="no"/>
@@
 <dimension x1="0" y1="63.49" x2="45.085" y2="63.5" x3="22.541934375" y3="66.034996875" textsize="1.778" layer="20" unit="inch" visible="yes"/>
 <dimension x1="0" y1="0" x2="0" y2="63.49" x3="-2.54" y3="31.745" textsize="1.778" layer="20" unit="inch" visible="yes"/>
+<text x="20.32" y="-6.985" size="1.778" layer="48" align="bottom-center">Released under Creative Commons license BY-SA 4.0
+https://creativecommons.org/licenses/by-sa/4.0</text>
 </plain>
 <attributes>
@@
 <pass name="Default">
 <param name="RoutingGrid" value="10mil"/>
+<param name="AutoGrid" value="1"/>
+<param name="Efforts" value="0"/>
+<param name="TopRouterVariant" value="1"/>
 <param name="tpViaShape" value="round"/>
 <param name="PrefDir.1" value="|"/>
