File: turbidity/devices/basic-handheld-turbidimeter/hardware/basic-handheld-turbidimeter.sch (EAGLE design)
At the start: 33 parts, among them Q1 16.000, U1 ATMEGA328P-PU

Commit message: updating pdfs of board and schematic
Other:
- note added: "Released under Creative Commons license BY-SA 4.0 https://creativecommons.org/licenses/by-sa/4.0"
- moved on the sheet: BTN, R8
Changed lines of the file:
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@@
 <?xml version="1.0" encoding="utf-8"?>
 <!DOCTYPE eagle SYSTEM "eagle.dtd">
-<eagle version="6.5.0">
+<eagle version="7.3.0">
 <drawing>
 <settings>
@@
 <part name="C6" library="SparkFun-Capacitors" deviceset="CAP" device="EZ" value="100nF"/>
 <part name="U$6" library="awqua_eagle_library" deviceset="AL5809" device=""/>
+<part name="FRAME1" library="frames" deviceset="DOCFIELD" device=""/>
 </parts>
 <sheets>
 <sheet>
 <plain>
+<text x="30.48" y="-2.54" size="1.778" layer="94">Released under Creative Commons license BY-SA 4.0
+https://creativecommons.org/licenses/by-sa/4.0</text>
 </plain>
 <instances>
@@
 <instance part="R6" gate="G$1" x="73.66" y="22.86" rot="R270"/>
 <instance part="R7" gate="G$1" x="55.88" y="20.32" rot="R180"/>
-<instance part="R8" gate="G$1" x="43.18" y="-7.62" rot="R270"/>
+<instance part="R8" gate="G$1" x="104.14" y="53.34" rot="R270"/>
 <instance part="C7" gate="G$1" x="-5.08" y="55.88" rot="R270"/>
 <instance part="C8" gate="G$1" x="0" y="60.96"/>
@@
 <attribute name="NAME" x="-27.94" y="72.39" size="1.778" layer="95"/>
 </instance>
-<instance part="BTN" gate="G$1" x="53.34" y="-2.54"/>
+<instance part="BTN" gate="G$1" x="114.3" y="58.42"/>
 <instance part="USB2SERIAL" gate="A" x="-25.4" y="15.24" rot="R180"/>
 <instance part="C9" gate="G$1" x="-12.7" y="20.32" smashed="yes" rot="R270">
@@
 <instance part="SUPPLY8" gate="GND" x="5.08" y="17.78"/>
 <instance part="SUPPLY10" gate="GND" x="-5.08" y="-20.32"/>
-<instance part="SUPPLY11" gate="GND" x="43.18" y="-17.78"/>
+<instance part="SUPPLY11" gate="GND" x="104.14" y="43.18"/>
 <instance part="SUPPLY9" gate="GND" x="2.54" y="22.86" rot="R270"/>
 <instance part="SUPPLY13" gate="GND" x="0" y="71.12" rot="R180"/>
@@
 <instance part="C6" gate="G$1" x="-5.08" y="43.18" rot="R270"/>
 <instance part="U$6" gate="G$1" x="-38.1" y="-17.78"/>
+<instance part="FRAME1" gate="G$1" x="25.4" y="-30.48"/>
 </instances>
 <busses>
@@
 <segment>
 <pinref part="BTN" gate="G$1" pin="1"/>
-<wire x1="50.8" y1="0" x2="35.56" y2="0" width="0.1524" layer="91"/>
-<label x="35.56" y="0" size="1.778" layer="95"/>
+<wire x1="111.76" y1="60.96" x2="96.52" y2="60.96" width="0.1524" layer="91"/>
+<label x="96.52" y="60.96" size="1.778" layer="95"/>
 </segment>
 <segment>
@@
 <pinref part="R8" gate="G$1" pin="2"/>
 <pinref part="SUPPLY11" gate="GND" pin="GND"/>
-<wire x1="43.18" y1="-15.24" x2="43.18" y2="-12.7" width="0.1524" layer="91"/>
+<wire x1="104.14" y1="45.72" x2="104.14" y2="48.26" width="0.1524" layer="91"/>
 </segment>
 <segment>
@@
 <pinref part="BTN" gate="G$1" pin="2"/>
 <pinref part="R8" gate="G$1" pin="1"/>
-<wire x1="50.8" y1="-2.54" x2="43.18" y2="-2.54" width="0.1524" layer="91"/>
-<wire x1="43.18" y1="-2.54" x2="35.56" y2="-2.54" width="0.1524" layer="91"/>
-<junction x="43.18" y="-2.54"/>
-<label x="35.56" y="-2.54" size="1.778" layer="95"/>
+<wire x1="111.76" y1="58.42" x2="104.14" y2="58.42" width="0.1524" layer="91"/>
+<wire x1="104.14" y1="58.42" x2="96.52" y2="58.42" width="0.1524" layer="91"/>
+<junction x="104.14" y="58.42"/>
+<label x="96.52" y="58.42" size="1.778" layer="95"/>
 </segment>
 <segment>
@@
 </schematic>
 </drawing>
+<compatibility>
+<note version="6.3" minversion="6.2.2" severity="warning">
+Since Version 6.2.2 text objects can contain more than one line,
+which will not be processed correctly with this version.
+</note>
+</compatibility>
 </eagle>
